File: stm-esc/stm-esc.kicad_pcb (KiCad board)
At the start: 2 copper layers, 40 x 80 mm, 41 parts, among them J1 RCP, J10 COUT, J2 Conn_01x06, J3 USART, J4 Conn_01x06, J5 SWIM, J6 AOUT, J7 CONN_01X01, J8 CONN_01X01, J9 BOUT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

Commit message: almost done for stm-esc
Parts:
- removed C6: C, Capacitors_SMD:C_0805
- C1: footprint Capacitors_THT:CP_Axial_L21.0mm_D8.0mm_P28.00mm_Horizontal -> Capacitors_SMD:C_0805
- U2: footprint TO_SOT_Packages_SMD:SOT-89-3 -> TO_SOT_Packages_SMD:SOT-89-3_Handsoldering
- moved R3 217.2 mm to (122.0, 136.7), turned to 180 degrees
- moved R1 207.6 mm to (121.1, 142.4), turned to 270 degrees
- moved R2 206.2 mm to (122.0, 138.1), turned to 180 degrees
- moved R4 205.5 mm to (122.0, 135.2)
- moved J10 204.6 mm to (107.7, 110.8)
- moved U2 204.5 mm to (110.2, 149.3), turned to 90 degrees
- moved R5 200.5 mm to (122.0, 139.6)
- moved U1 198.1 mm to (119.3, 149.3)
- moved R6 196.2 mm to (122.6, 142.4), turned to 90 degrees
- moved R10 186.0 mm to (125.0, 141.1)
- moved U3 184.5 mm to (113.7, 135.8), turned to 90 degrees
- moved R7 184.5 mm to (125.0, 135.2)
- moved R9 183.8 mm to (125.0, 139.6)
- moved R8 183.0 mm to (125.0, 137.4)
- moved C1 178.5 mm to (105.6, 143.9), turned to 270 degrees
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Connections:
- C1 pad 1: VCC -> /RCP
- C1 pad 2: GND -> Net-(C1-Pad2)
- C2 pad 1: /RCP -> +3V3
- C2 pad 2: Net-(C2-Pad2) -> GND
- C3 pad 1: +3V3 -> Net-(C3-Pad1)
- C3 pad 2: GND -> AOUT
- C4 pad 2: AOUT -> BOUT
- C5 pad 2: BOUT -> COUT
- D1 pad 1: Net-(C4-Pad1) -> Net-(C3-Pad1)
- D2 pad 1: Net-(C5-Pad1) -> Net-(C4-Pad1)
- D3 pad 1: Net-(C6-Pad1) -> Net-(C5-Pad1)
- J1 pad 1: Net-(C2-Pad2) -> Net-(C1-Pad2)
- J4 pad 1: Net-(J4-Pad1) -> GND
- U3 pad 23: /SWDIO -> /SWCLK
- U3 pad 24: /SWCLK -> /SWDIO
- U4 pad 8: Net-(C4-Pad1) -> Net-(C3-Pad1)
- U5 pad 8: Net-(C5-Pad1) -> Net-(C4-Pad1)
- U6 pad 8: Net-(C6-Pad1) -> Net-(C5-Pad1)
Routing:
- net VCC: track 0.00 -> 54.5 mm
- net AOUT: track 0.00 -> 49.5 mm, vias 0 -> 3
- net BOUT: track 0.00 -> 45.1 mm, vias 0 -> 3
- net COUT: track 0.00 -> 45.0 mm, vias 0 -> 3
- net +5V: track 0.00 -> 44.3 mm
- net +3V3: track 0.00 -> 29.4 mm, vias 0 -> 1
- net GND: track 0.00 -> 26.9 mm, vias 0 -> 18
- net Net-(Q2-Pad4): track 0.00 -> 26.0 mm, vias 0 -> 2
- net Net-(Q4-Pad4): track 0.00 -> 25.8 mm, vias 0 -> 2
- net Net-(Q6-Pad4): track 0.00 -> 25.6 mm, vias 0 -> 2
- net /Fabc-: track 0.00 -> 18.4 mm
- net CP: track 0.00 -> 16.9 mm, vias 0 -> 2
- net Net-(C3-Pad1): track 0.00 -> 16.4 mm, vias 0 -> 2
- net AN: track 0.00 -> 15.5 mm
- net AP: track 0.00 -> 15.0 mm, vias 0 -> 2
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- added copper zone on F.Cu, net AOUT
- added copper zone on F.Cu, net BOUT
- added copper zone on F.Cu, net COUT
- added copper zone on B.Cu, net GND
- added copper zone on F.Cu, net GND
Other:
- board size 40 x 80 mm -> 40 x 60 mm

Commit message: improve
Parts:
- moved J7 140.8 mm to (23.1, 35.4)
- moved J8 138.6 mm to (23.1, 23.3)
- moved J2 121.9 mm to (40.7, 65.0), turned to 0 degrees
- moved R9 118.9 mm to (47.6, 49.3)
- moved R5 118.7 mm to (45.0, 49.3)
- moved J1 116.6 mm to (23.1, 59.7)
- moved R2 116.5 mm to (44.9, 50.8)
- moved J5 115.9 mm to (23.1, 50.9)
- moved R1 115.7 mm to (44.9, 55.3), turned to 180 degrees
- moved C1 115.6 mm to (25.7, 60.3)
- moved R6 115.6 mm to (44.9, 56.8), turned to 0 degrees
- moved R8 115.0 mm to (47.6, 52.3)
- moved R10 114.4 mm to (47.7, 56.8)
- moved R3 114.3 mm to (44.9, 52.2)
- moved U6 113.8 mm to (30.6, 41.5)
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Connections:
- J2 pad 1: /NRST -> /PB3
- J2 pad 2: /PF1 -> /PA12
- J2 pad 3: /PF0 -> /PA11
- J2 pad 4: /PB5 -> /PB4
- J2 pad 5: /PB4 -> /PB5
- J2 pad 6: /PB3 -> /PA6
- J3 pad 1: /RXD -> /TXD
- J3 pad 2: /TXD -> /RXD
- J4 pad 1: GND -> /PA3
- J4 pad 2: /PA12 -> /PA2
- J4 pad 3: /PA11 -> /NRST
- J4 pad 4: /PA6 -> /PF1
- J4 pad 5: /PA3 -> /PF0
- J4 pad 6: /PA2 -> GND
Routing:
- net GND: track 26.9 -> 57.1 mm, vias 18 -> 28
- net /PA2: track 2.28 -> 30.8 mm
- net /PF0: track 1.96 -> 28.9 mm
- net /PA3: track 2.22 -> 29.1 mm
- net /PF1: track 1.95 -> 28.5 mm
- net /NRST: track 1.93 -> 28.2 mm
- net AN: track 15.5 -> 40.5 mm
- net /PA6: track 1.55 -> 25.0 mm
- net +5V: track 44.3 -> 64.6 mm
- net +3V3: track 29.4 -> 49.3 mm, vias 1 -> 3
- net BN: track 6.73 -> 26.1 mm
- net /PB5: track 1.43 -> 20.1 mm
- net AP: track 15.0 -> 31.8 mm
- net /PB4: track 1.43 -> 15.2 mm
- net /PA11: track 1.46 -> 15.1 mm
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Other:
- board size 40 x 60 mm -> 57 x 48 mm
- board text added: "B3 A12 A11 B4 B5 A6 A3 A2 RST F1 F0"
- board text added: "DIO CLK"
- board text added: "TXD RXD"

Commit message: 定板打样stm-esc
Parts:
- removed U1: LM78M05CT, TO_SOT_Packages_SMD:TO-252-2
- U2: footprint TO_SOT_Packages_SMD:SOT-89-3_Handsoldering -> TO_SOT_Packages_SMD:SOT-223-3_TabPin2
- moved U2 5.90 mm to (56.5, 51.3)
Connections:
- J1 pad 2: +5V -> +3V3
- J3 pad 4: +5V -> +3V3
- U2 pad 3: +5V -> VCC
Routing:
- net +5V: track 64.6 -> 0.00 mm
- net +3V3: track 49.3 -> 98.0 mm, vias 3 -> 2
- net GND: track 57.1 -> 66.1 mm, vias 28 -> 42
- net VCC: track 67.6 -> 65.7 mm
- net BP: track 15.4 -> 16.6 mm
- net AP: track 31.8 -> 32.7 mm
- net COUT: track 39.9 -> 40.4 mm
