File: timer/timer.kicad_pcb (KiCad board)
At the start: 2 copper layers, 90 x 90 mm, 45 parts, among them J1 Conn_01x02, J2 Conn_Coaxial, J3 Conn_01x04, J4 Conn_01x04, J5 Conn_01x04, J8 Conn_01x02, Q1 2N7002, Q2 nfet, SW1 Rotary_Encoder_Switch, U1 AMS1117-3.3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

Commit message: working
Parts:
- removed B+, B-: Conn_01x01, Connector_Wire:SolderWirePad_1x01_Drill2.5mm
- added D2: D, Diode_SMD:D_0603_1608Metric_Pad1.05x0.95mm_HandSolder, F.Cu at (29.5, 61.6)
- added J6: GND/B-, Connector_Wire:SolderWirePad_1x01_Drill2.5mm, F.Cu at (24.9, 105.4)
- added J7: Conn_01x01, Connector_Wire:SolderWirePad_1x01_Drill2.5mm, F.Cu at (24.5, 89.2)
- added Q3: nfet, footprint:SOIC-8, F.Cu at (86.0, 77.3)
- added R20: 0.1r, Resistor_THT:R_Axial_DIN0918_L18.0mm_D9.0mm_P22.86mm_Horizontal, F.Cu at (103.9, 83.8)
- added R21: 1k, Resistor_SMD:R_0603_1608Metric_Pad1.05x0.95mm_HandSolder, F.Cu at (78.5, 61.2)
- added SW2: SW_DIP_x01, Button_Switch_SMD:SW_SPST_CK_RS282G05A3, F.Cu at (24.0, 25.6)
- C8: value Cvs -> Cbs
- J1: value Conn_01x02 -> Conn_01x01; footprint Connector_PinHeader_2.54mm:PinHeader_1x02_P2.54mm_Vertical -> Connector_Wire:SolderWirePad_1x01_Drill2.5mm
- J2: value Conn_Coaxial -> Conn_01x01; footprint Connector_Coaxial:SMA_Amphenol_132289_EdgeMount -> Connector_Wire:SolderWirePad_1x01_Drill2.5mm
- J8: moved to B.Cu
- Q1: value 2N7002 -> Q_NPN_BEC
- Q2: value nfet -> 2N7002; footprint footprint:SOIC-8 -> Package_TO_SOT_SMD:SOT-23
- R12, R13: value 10k -> 1k
- U1: value AMS1117-3.3 -> REGULAR-7133-1; footprint Package_TO_SOT_SMD:SOT-223-3_TabPin2 -> Package_TO_SOT_SMD:SOT-89-3_Handsoldering
- moved D1 89.2 mm to (22.7, 69.4)
- moved R1 88.7 mm to (23.6, 65.8), turned to 0 degrees
- moved R4 80.2 mm to (27.7, 49.0), turned to 0 degrees
- moved R5 80.2 mm to (27.7, 51.7), turned to 0 degrees
- moved J2 72.8 mm to (33.7, 105.5)
- moved U1 58.3 mm to (48.2, 68.7), turned to 180 degrees
- moved R17 57.0 mm to (91.9, 83.8), turned to 270 degrees
- moved R13 54.2 mm to (86.1, 65.6), turned to 270 degrees
- moved R12 53.7 mm to (89.0, 65.7)
- moved BZ1 48.8 mm to (62.8, 65.4), turned to 0 degrees
- moved J1 47.6 mm to (24.3, 80.1)
- moved R18 43.5 mm to (43.9, 83.8), turned to 270 degrees
- moved R19 42.5 mm to (67.9, 106.6), turned to 90 degrees
- moved Q2 42.2 mm to (76.7, 64.4), turned to 270 degrees
- moved R16 42.1 mm to (79.9, 106.6), turned to 90 degrees
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Connections:
- J1 pad 1: GND -> VCC
- J2 pad 1: VCC -> GND
- Q1 pad 1: Beep -> Net-(Q1-Pad1)
- Q1 pad 3: Net-(BZ1-Pad2) -> Net-(Q1-Pad3)
- Q2 pad 1: B- -> Net-(Q2-Pad1)
- Q2 pad 2: B- -> GND
- Q2 pad 3: B- -> Net-(BZ1-Pad2)
- R12 pad 1: Net-(Q2-Pad4) -> Net-(Q1-Pad1)
- R13 pad 2: Net-(Q2-Pad4) -> Net-(Q1-Pad3)
- R14 pad 1: B- -> Net-(Q3-Pad1)
- R16 pad 2: Net-(Q2-Pad5) -> Net-(Q3-Pad5)
- R17 pad 1: B- -> Net-(Q3-Pad1)
- R19 pad 2: Net-(Q2-Pad5) -> Net-(Q3-Pad5)
- R3 pad 2: +3V3 -> Net-(D2-Pad1)
- U1 pad 2: +3V3 -> VCC
- U1 pad 3: VCC -> +3V3
- U2 pad 1: +3V3 -> +1V5
Routing:
- net /RESET: track 63.5 -> 0.00 mm, vias 2 -> 0
- net GND: track 25.2 -> 82.3 mm, vias 1 -> 0
- net /SWDIO: track 51.7 -> 0.00 mm
- net Net-(Q3-Pad1): track 0.00 -> 47.8 mm
- net /SWCLK: track 44.9 -> 0.00 mm
- net Discharge: track 0.00 -> 42.5 mm, vias 0 -> 2
- net +3V3: track 40.6 -> 0.00 mm
- net B+: track 71.3 -> 33.7 mm
- net Net-(DS1-Pad14): track 28.8 -> 0.00 mm, vias 1 -> 0
- net Net-(DS1-Pad4): track 26.8 -> 0.00 mm, vias 1 -> 0
- net Net-(DS1-Pad5): track 23.6 -> 0.00 mm, vias 1 -> 0
- net Net-(DS1-Pad12): track 22.2 -> 0.00 mm, vias 1 -> 0
- net Net-(DS1-Pad13): track 22.2 -> 0.00 mm, vias 1 -> 0
- net Net-(DS1-Pad6): track 20.7 -> 0.00 mm, vias 1 -> 0
- net Net-(DS1-Pad11): track 20.6 -> 0.00 mm, vias 1 -> 0
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- added copper zone on F.Cu, net Net-(Q3-Pad1)
- added copper zone on F.Cu, net Net-(Q3-Pad5)
